File: Atari2600_2TransistorCompMod.kicad_sch (KiCad schematic)
At the start: 15 parts, among them J1 RFModulatorHeader, J2 AudioIn, J3 CompositeOut, Q1 MMBT3904, Q2 MMBT3906

Commit message: Added gerbers and iBOM
Other:
- title: (none) -> Atari2600_2TransistorCompMod
Changed lines of the file:
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@@
 	(generator_version "9.0")
 	(paper "A4")
+	(title_block
+		(title "Atari2600_2TransistorCompMod")
+	)
 	(junction
 		(at 41.91 53.34)
